Commit message: arm position on table

File: panda_description/urdf/CamToHand.xacro (robot description, xacro)
@@ -89,5 +89,5 @@
     <parent link="world"/>
     <child link="link_1"/>
-    <origin xyz="0 0 ${length1/2}" rpy="0 0 0"/>
+    <origin xyz="0 1 ${length1/2}" rpy="0 0 0"/>
   </joint>
   <joint name="pan_joint" type="continuous">

File: panda_description/urdf/panda.urdf.xacro (robot description, xacro)
@@ -7,4 +7,5 @@
   <xacro:include filename="$(find panda_description)/urdf/panda_arm.xacro" />
   <xacro:include filename="$(find panda_description)/urdf/panda_gripper.xacro" />
+  <!-- <xacro:include filename="$(find panda_description)/urdf/CamToHand.xacro" /> -->
   <xacro:include filename="$(find panda_description)/urdf/panda_utils.xacro" />
   <!--            -->

File: panda_description/urdf/panda_arm.xacro (robot description, xacro)
@@ -12,5 +12,5 @@
   <xacro:arg name="add_plug" default="false" />
   <xacro:arg name="use_mesh" default="true" />
-  <xacro:include filename="$(find realsense2_description)/urdf/_d435.urdf.xacro" />
+  <!-- <xacro:include filename="$(find realsense2_description)/urdf/_d435.urdf.xacro" /> -->
   <!--            -->
   <!-- Properties -->
@@ -352,5 +352,5 @@
     panda_moveit_config)/config/initial_positions.yaml"/>
     -->
-    <xacro:sensor_d435 parent="${prefix}${link0_name}"
+    <!-- <xacro:sensor_d435 parent="${prefix}${link0_name}"
       use_nominal_extrinsics="$(arg use_nominal_extrinsics)" add_plug="$(arg add_plug)"
       use_mesh="$(arg use_mesh)">
@@ -408,5 +408,5 @@
         </plugin>
       </sensor>
-    </gazebo>
+    </gazebo> -->
     <ros2_control name="2DofPosition" type="gz_ros2_control/GazeboSimSystem">
       <hardware>

Commit message: added sensor pole

File: panda_description/urdf/CamToHand.xacro (robot description, xacro)
@@ -1,99 +1,112 @@
 <?xml version="1.0"?>
-<robot name="sensor_stick" xmlns:xacro="http://www.ros.org/wiki/xacro">
-  <!--Define constants-->
-  <xacro:property name="PI" value="3.14159"/>
+<robot xmlns:xacro="http://wiki.ros.org/xacro" name="PoleSensor">
+  <!-- <robot  xmlns:xacro="http://www.ros.org/wiki/xacro"> -->
+  <!--Define
+  constants-->
+  <xacro:property name="PI" value="3.14159" />
   <xacro:property name="mass1" value="10" />
   <xacro:property name="mass2" value="1" />
-  <xacro:property name="width1" value="0.1" /> <!--link_1 radius-->
-  <xacro:property name="width2" value="0.1" /> <!--link_2 radius-->
-  <xacro:property name="length0" value="0.1" /> <!--link_1 length-->
-  <xacro:property name="length1" value="1.5" /> <!--link_2 length-->
-  <xacro:property name="length2" value="0.1" /> <!--link_3 length-->
+  <xacro:property name="width1" value="0.1" /> <!--link_1
+  radius-->
+  <xacro:property name="width2" value="0.1" /> <!--link_2
+  radius-->
+  <xacro:property name="length0" value="0.1" /> <!--link_1
+  length-->
+  <xacro:property name="length1" value="1.5" /> <!--link_2
+  length-->
+  <xacro:property name="length2" value="0.1" /> <!--link_3
+  length-->
+  <xacro:property name="Custom_length" value="0.275935" /> <!--link_3
+  length-->
   <xacro:property name="mass_camera" value="0.2" />
-  <!--Import gazebo elements-->
-  <xacro:include filename="/home/akhil/panda_arm/panda_description/urdf/sensor_stick.gazebo.xacro" />
-  <!--Links-->
-  <link name="world"/>
+  <!--Import
+  gazebo elements-->
+  <!-- <xacro:include
+  filename="/home/akhil/panda_arm/panda_description/urdf/sensor_stick.gazebo.xacro" /> -->
+  <xacro:include filename="$(find panda_description)/urdf/sensor_stick.gazebo.xacro" />
+  <!-- Links -->
+  <link name="world" />
   <link name="link_1">
     <visual>
-      <origin xyz="0 0 0" rpy="0 0 0"/>
+      <origin xyz="0 0 0" rpy="0 0 0" />
       <geometry>
-        <box size="${width1} ${width1} ${length1}"/>
+        <box size="${width1} ${width1} ${length1}" />
       </geometry>
       <material name="blue">
-        <color rgba="0.0 0.0 0.8 1.0"/>
+        <color rgba="0.0 0.0 0.8 1.0" />
       </material>
     </visual>
     <collision>
-      <origin xyz="0 0 0" rpy="0 0 0"/>
+      <origin xyz="0 0 0" rpy="0 0 0" />
       <geometry>
-        <box size="${width1} ${width1} ${length1}"/>
+        <box size="${width1} ${width1} ${length1}" />
       </geometry>
     </collision>
     <inertial>
-      <origin xyz="0 0 0" rpy="0 0 0"/>
-      <mass value="${mass1}"/>
+      <origin xyz="0 0 0" rpy="0 0 0" />
+      <mass value="${mass1}" />
       <inertia
         ixx="${mass1 / 12.0 * (width1*width1 + length1*length1)}" ixy="0.0" ixz="0.0"
         iyy="${mass1 / 12.0 * (length1*length1 + width1*width1)}" iyz="0.0"
-        izz="${mass1 / 12.0 * (width1*width1 + width1*width1)}"/>
+        izz="${mass1 / 12.0 * (width1*width1 + width1*width1)}" />
     </inertial>
   </link>
   <link name="link_2">
     <visual>
-      <origin xyz="0 0 0" rpy="0 0 0"/>
+      <origin xyz="0 0 0" rpy="0 0 0" />
       <geometry>
-        <box size="${width2} ${width2} ${length2}"/>
+        <box size="${width2} ${width2} ${length2}" />
       </geometry>
       <material name="white">
-        <color rgba="1.0 1.0 1.0 1.0"/>
+        <color rgba="1.0 1.0 1.0 1.0" />
       </material>
     </visual>
     <collision>
-      <origin xyz="0 0 0" rpy="0 0 0"/>
+      <origin xyz="0 0 0" rpy="0 0 0" />
       <geometry>
-        <box size="${width2} ${width2} ${length2}"/>
+        <box size="${width2} ${width2} ${length2}" />
       </geometry>
     </collision>
     <inertial>
-      <origin xyz="0 0 0" rpy="0 0 0"/>
-      <mass value="${mass2}"/>
+      <origin xyz="0 0 0" rpy="0 0 0" />
+      <mass value="${mass2}" />
       <inertia
         ixx="${mass2 / 12.0 * (width2*width2 + length2*length2)}" ixy="0.0" ixz="0.0"
         iyy="${mass2 / 12.0 * (length2*length2 + width2*width2)}" iyz="0.0"
-        izz="${mass2 / 12.0 * (width2*width2 + width2*width2)}"/>
+        izz="${mass2 / 12.0 * (width2*width2 + width2*width2)}" />
     </inertial>
   </link>
   <!-- RGBD camera -->
   <link name="camera_link">
-  <collision>
-    <origin xyz="-0.016 0 0" rpy="0 0 0"/>
-    <geometry>
-      <box size="0.036 0.18 0.04"/>
-    </geometry>
-  </collision>
-  <visual>
-    <origin xyz="0 0 0" rpy="0 0 0"/>
-    <geometry>
-      <mesh filename="package://panda_description/meshes/visual/asus_xtion.dae"/>
-    </geometry>
-  </visual>
-  <inertial>
-    <mass value="${mass_camera}" />
-    <origin xyz="0 0 0" rpy="0 0 0"/>
-    <inertia ixx="5.8083e-4" ixy="0" ixz="0" iyy="3.0833e-5" iyz="0" izz="5.9083e-4" />
-  </inertial>
+    <collision>
+      <origin xyz="-0.016 0 0" rpy="0 0 0" />
+      <geometry>
+        <box size="0.036 0.18 0.04" />
+      </geometry>
+    </collision>
+    <visual>
+      <origin xyz="0 0 0" rpy="0 0 0" />
+      <geometry>
+        <mesh filename="package://panda_description/meshes/visual/asus_xtion.dae" />
+      </geometry>
+    </visual>
+    <inertial>
+      <mass value="${mass_camera}" />
+      <origin xyz="0 0 0" rpy="0 0 0" />
+      <inertia ixx="5.8083e-4" ixy="0" ixz="0" iyy="3.0833e-5" iyz="0" izz="5.9083e-4" />
+    </inertial>
   </link>
   <!--Joints-->
   <joint name="fixed_base_joint" type="fixed">
-    <parent link="world"/>
-    <child link="link_1"/>
-    <origin xyz="0 1 ${length1/2}" rpy="0 0 0"/>
+    <parent link="world" />
+    <child link="link_1" />
+    <origin xyz="0 -2 -${Custom_length}" rpy="0 0 0" />
   </joint>
   <joint name="pan_joint" type="continuous">
-    <parent link="link_1"/>
-    <child link="link_2"/>
-    <axis xyz="0 0 1"/>
-    <origin xyz="0 0 ${length1/2+length2/2}" rpy="0 0 -${pi/2}"/>
+    <parent link="link_1" />
+    <child link="link_2" />
+    <axis xyz="0 0 1" />
+    <!-- <origin xyz="0 0 ${length1/2+length2/2}" rpy="0 0 ${pi/2}"/> -->
+    <origin xyz="0 0 ${length1/2+length2/2}" rpy="0 0 ${PI/2}" />
   </joint>
   <joint name="tilt_joint" type="continuous">
@@ -101,5 +114,5 @@
     <parent link="link_2" />
     <child link="camera_link" />
-    <axis xyz="0 1 0"/>
+    <axis xyz="0 1 0" />
   </joint>
   <link name="camera_rgb_frame" />
@@ -127,24 +140,3 @@
     <child link="camera_depth_optical_frame" />
   </joint>
-  <!--Transmission and actuators-->
-  <transmission name="tran1">
-    <type>transmission_interface/SimpleTransmission</type>
-    <joint name="pan_joint">
-      <hardwareInterface>hardware_interface/PositionJointInterface</hardwareInterface>
-    </joint>
-    <actuator name="motor1">
-      <hardwareInterface>hardware_interface/PositionJointInterface</hardwareInterface>
-      <mechanicalReduction>1</mechanicalReduction>
-    </actuator>
-  </transmission>
-  <transmission name="tran2">
-    <type>transmission_interface/SimpleTransmission</type>
-    <joint name="tilt_joint">
-      <hardwareInterface>hardware_interface/PositionJointInterface</hardwareInterface>
-    </joint>
-    <actuator name="motor2">
-      <hardwareInterface>hardware_interface/PositionJointInterface</hardwareInterface>
-      <mechanicalReduction>1</mechanicalReduction>
-    </actuator>
-  </transmission>
 </robot>

File: panda_description/urdf/panda.urdf.xacro (robot description, xacro)
@@ -7,5 +7,4 @@
   <xacro:include filename="$(find panda_description)/urdf/panda_arm.xacro" />
   <xacro:include filename="$(find panda_description)/urdf/panda_gripper.xacro" />
-  <!-- <xacro:include filename="$(find panda_description)/urdf/CamToHand.xacro" /> -->
   <xacro:include filename="$(find panda_description)/urdf/panda_utils.xacro" />
   <!--            -->
@@ -37,5 +36,5 @@
   <xacro:arg name="ros2_control_command_interface" default="position" />
   <!-- The filepath to parameters of ROS 2 controllers
-  <xacro:arg name="ros2_controller_parameters" default="$(find
+  <xacro:arg name="ros2_controller_parameters" defaulst="$(find
   panda_description)/config/controllers_$(arg ros2_control_command_interface).yaml"/>
   -->

File: panda_description/urdf/sensor_stick.gazebo.xacro (robot description, xacro)
@@ -1,72 +1,69 @@
 <?xml version="1.0"?>
 <robot>
-  <!-- ros_control plugin -->
-  <gazebo>
-    <plugin name="gazebo_ros_control" filename="libgazebo_ros_control.so">
-      <robotNamespace>/sensor_stick</robotNamespace>
-      <robotSimType>gazebo_ros_control/DefaultRobotHWSim</robotSimType>
-    </plugin>
-  </gazebo>
-  <!--base_link-->
   <gazebo reference="base_link">
     <material>Gazebo/White</material>
   </gazebo>
-  <!--link_1-->
   <gazebo reference="link_1">
-    <mu1>0.2</mu1>
-    <mu2>0.2</mu2>
     <material>Gazebo/Orange</material>
+    <surface>
+      <friction>
+        <ode>
+          <mu>0.2</mu>
+          <mu2>0.2</mu2>
+        </ode>
+      </friction>
+    </surface>
   </gazebo>
-  <!--link_2-->
   <gazebo reference="link_2">
-    <mu1>0.2</mu1>
-    <mu2>0.2</mu2>
     <material>Gazebo/White</material>
+    <surface>
+      <friction>
+        <ode>
+          <mu>0.2</mu>
+          <mu2>0.2</mu2>
+        </ode>
+      </friction>
+    </surface>
   </gazebo>
-  <!--camera_link-->
   <gazebo reference="camera_link">
-    <mu1>0.2</mu1>
-    <mu2>0.2</mu2>
     <material>Gazebo/Grey</material>
+    <surface>
+      <friction>
+        <ode>
+          <mu>0.2</mu>
+          <mu2>0.2</mu2>
+        </ode>
+      </friction>
+    </surface>
   </gazebo>
-  <!--RGBD camera -->
   <gazebo reference="camera_rgb_frame">
-   <sensor type="depth" name="camera">
-     <always_on>true</always_on>
-     <visualize>false</visualize>
-     <update_rate>15.0</update_rate>
-     <camera name="front">
-       <horizontal_fov>1.047197</horizontal_fov>
-       <image>
-         <!-- openni_kinect plugin works only with BGR8 -->
-         <format>B8G8R8</format>
-         <width>640</width>
-         <height>480</height>
-       </image>
-       <clip>
-         <near>0.01</near>
-         <far>9</far>
-       </clip>
-     </camera>
-     <plugin name="camera_controller" filename="libgazebo_ros_openni_kinect.so">
-       <baseline>0.1</baseline>
-       <alwaysOn>true</alwaysOn>
-       <updateRate>15.0</updateRate>
-       <cameraName>camera</cameraName>
-       <imageTopicName>/camera/rgb/image_raw</imageTopicName>
-       <cameraInfoTopicName>/camera/rgb/camera_info</cameraInfoTopicName>
-       <depthImageTopicName>/camera/depth_registered/image_raw</depthImageTopicName>
-       <depthImageCameraInfoTopicName>/camera/depth_registered/camera_info</depthImageCameraInfoTopicName>
-       <pointCloudTopicName>/camera/depth_registered/points</pointCloudTopicName>
-       <frameName>camera_rgb_optical_frame</frameName>
-       <pointCloudCutoff>0.35</pointCloudCutoff>
-       <pointCloudCutoffMax>4.5</pointCloudCutoffMax>
-       <CxPrime>0</CxPrime>
-       <Cx>0</Cx>
-       <Cy>0</Cy>
-       <focalLength>0</focalLength>
-       <hackBaseline>0</hackBaseline>
-     </plugin>
-   </sensor>
+    <sensor type="rgbd_camera" name="sensor_pole_rgbd_camera">
+      <always_on>true</always_on>
+      <visualize>false</visualize> <update_rate>15</update_rate>
+      <camera name="color_camera">
+        <horizontal_fov>1.047</horizontal_fov>
+        <image>
+          <width>640</width>
+          <height>480</height>
+          <format>R8G8B8</format> </image>
+        <clip>
+          <near>0.01</near>
+          <far>9</far>
+        </clip>
+        <topic>/color_camera</topic>
+      </camera>
+      <depth_camera name="depth_camera">
+        <image>
+          <topic>/depth_camera</topic>
+        </image>
+        <point_cloud>
+          <topic>/depth_camera/points</topic>
+        </point_cloud>
+        <clip>
+          <near>0.01</near>
+          <far>9</far>
+        </clip>
+      </depth_camera>
+    </sensor>
   </gazebo>
 </robot>
