Commit message: saparate sensor roboModel

File: panda_description/urdf/panda_arm.xacro (robot description, xacro)
@@ -355,5 +355,5 @@
       use_nominal_extrinsics="$(arg use_nominal_extrinsics)" add_plug="$(arg add_plug)"
       use_mesh="$(arg use_mesh)">
-      <origin xyz="0.1 0.0 0.05" rpy="0 0.0 0" />
+      <origin xyz="0.8 0.0 0.05" rpy="0 0.0 0" />
     </xacro:sensor_d435>
     <gazebo reference="${prefix}${link0_name}">

File: panda_description/urdf/sensor_stick.gazebo.xacro (robot description, xacro)
@@ -1,69 +1,58 @@
 <?xml version="1.0"?>
 <robot>
-  <gazebo reference="base_link">
-    <material>Gazebo/White</material>
-  </gazebo>
-  <gazebo reference="link_1">
-    <material>Gazebo/Orange</material>
-    <surface>
-      <friction>
-        <ode>
-          <mu>0.2</mu>
-          <mu2>0.2</mu2>
-        </ode>
-      </friction>
-    </surface>
-  </gazebo>
-  <gazebo reference="link_2">
-    <material>Gazebo/White</material>
-    <surface>
-      <friction>
-        <ode>
-          <mu>0.2</mu>
-          <mu2>0.2</mu2>
-        </ode>
-      </friction>
-    </surface>
-  </gazebo>
-  <gazebo reference="camera_link">
-    <material>Gazebo/Grey</material>
-    <surface>
-      <friction>
-        <ode>
-          <mu>0.2</mu>
-          <mu2>0.2</mu2>
-        </ode>
-      </friction>
-    </surface>
-  </gazebo>
-  <gazebo reference="camera_rgb_frame">
-    <sensor type="rgbd_camera" name="sensor_pole_rgbd_camera">
-      <always_on>true</always_on>
-      <visualize>false</visualize> <update_rate>15</update_rate>
-      <camera name="color_camera">
-        <horizontal_fov>1.047</horizontal_fov>
-        <image>
-          <width>640</width>
-          <height>480</height>
-          <format>R8G8B8</format> </image>
-        <clip>
-          <near>0.01</near>
-          <far>9</far>
-        </clip>
+  <gazebo reference="link_1"><material>Gazebo/Orange</material></gazebo>
+  <gazebo reference="link_2"><material>Gazebo/White</material></gazebo>
+  <gazebo reference="camera_base_link"><material>Gazebo/Grey</material></gazebo>
+  <gazebo reference="camera_mount_link">
+      <sensor name="d435_color" type="camera">
+        <always_on>1</always_on>
+        <update_rate>30</update_rate>
+        <visualize>1</visualize>
+        <pose>0 0.0175 0.0 0 -0 0</pose>
         <topic>/color_camera</topic>
-      </camera>
-      <depth_camera name="depth_camera">
-        <image>
-          <topic>/depth_camera</topic>
-        </image>
-        <point_cloud>
-          <topic>/depth_camera/points</topic>
-        </point_cloud>
-        <clip>
-          <near>0.01</near>
-          <far>9</far>
-        </clip>
-      </depth_camera>
-    </sensor>
-  </gazebo>
+        <camera name="d435">
+          <horizontal_fov>1.21126</horizontal_fov>
+          <image>
+            <width>640</width>
+            <height>480</height>
+            <format>RGB_INT8</format>
+          </image>
+          <clip>
+            <near>0.1</near>
+            <far>100</far>
+          </clip>
+          <noise>
+            <type>gaussian</type>
+            <mean>0</mean>
+            <stddev>0.007</stddev>
+          </noise>
+        </camera>
+      </sensor>
+      <sensor name='d435_depth' type='depth_camera'>
+        <always_on>1</always_on>
+        <update_rate>15</update_rate>
+        <visualize>1</visualize>
+        <topic>/depth_camera</topic>
+        <pose>0 0.04 -0.04 0 0 0</pose>
+        <camera name='d435'>
+          <horizontal_fov>1.48702</horizontal_fov>
+          <image>
+            <width>1280</width>
+            <height>720</height>
+          </image>
+          <clip>
+            <near>0.2</near>
+            <far>5</far>
+          </clip>
+          <noise>
+            <type>gaussian</type>
+            <mean>0</mean>
+            <stddev>0.1</stddev>
+          </noise>
+        </camera>
+        <plugin filename="libgz-sim-sensors-system.so" name="gz::sim::systems::Sensors">
+          <render_engine>ogre</render_engine>
+        </plugin>
+      </sensor>
+    </gazebo>
 </robot>
