Commit message: Fixed sensor pole

File: panda_description/urdf/PoleSensor.urdf.xacro (robot description, xacro)
@@ -9,5 +9,5 @@
   <xacro:property name="length2" value="0.1" />
   <xacro:property name="Custom_length" value="0.275935" />
-  <xacro:include filename="$(find realsense2_description)/urdf/_d435.urdf.xacro" />
+  <!-- <xacro:include filename="$(find realsense2_description)/urdf/_d435.urdf.xacro" /> -->
   <xacro:include filename="$(find panda_description)/urdf/sensor_stick.gazebo.xacro" />
   <link name="world" />
@@ -38,9 +38,27 @@
     </inertial>
   </link>
-  <link name="camera_mount_link">
+   <link name='camera_link'>
+    <pose>0 0 0 0 0 0</pose>
     <inertial>
-      <mass value="0.001" />
-      <inertia ixx="0.0001" ixy="0" ixz="0" iyy="0.0001" iyz="0" izz="0.0001" />
+      <mass value="0.1"/>
+      <origin xyz="0 0 0" rpy="0 0 0"/>
+      <inertia
+          ixx="1e-6" ixy="0" ixz="0"
+          iyy="1e-6" iyz="0"
+          izz="1e-6"
+      />
     </inertial>
+    <collision name='collision'>
+      <origin xyz="0 0 0" rpy="0 0 0"/>
+      <geometry>
+        <box size=".03 .03 .03"/>
+      </geometry>
+    </collision>
+    <visual name='camera_link_visual'>
+      <origin xyz="0 0 0" rpy="0 0 0"/>
+      <geometry>
+        <box size=".03 .03 .03"/>
+      </geometry>
+    </visual>
   </link>
   <joint name="fixed_base_joint" type="fixed">
@@ -58,39 +76,18 @@
     <origin xyz="0.05 0 ${length2/2+0.02}" rpy="0 0.5 0" />
     <parent link="link_2" />
-    <child link="camera_mount_link" />
+    <child link="camera_link" />
     <axis xyz="0 1 0" />
   </joint>
- <xacro:sensor_d435 parent="camera_mount_link"
+ <!-- <xacro:sensor_d435 parent="camera_mount_link"
       use_nominal_extrinsics="true" add_plug="false"
       use_mesh="true">
       <origin xyz="0.8 0.0 0.05" rpy="0 0.0 0" />
-    </xacro:sensor_d435>
-<!--
-  <joint name="camera_base_mount_joint" type="fixed">
-    <parent link="camera_mount_link" />
-    <child link="camera_link" />
-    <origin xyz="0 0 0" rpy="0 0 0" />
+    </xacro:sensor_d435> -->
+ <joint type="fixed" name="camera_optical_joint">
+    <origin xyz="0 0 0" rpy="-1.5707 0 -1.5707"/>
+    <child link="camera_link_optical"/>
+    <parent link="camera_link"/>
   </joint>
-  <link name="camera_color_optical_frame">
-    <inertial>
-      <mass value="0.001" />
-      <inertia ixx="0.0001" ixy="0" ixz="0" iyy="0.0001" iyz="0" izz="0.0001" />
-    </inertial>
+  <link name="camera_link_optical">
   </link>
-  <joint name="camera_color_optical_joint" type="fixed">
-    <parent link="camera_link" />
-    <child link="camera_color_optical_frame" />
-    <origin xyz="0 0.01 0" rpy="-1.570796 0 -1.570796" />
-  </joint>
-  <link name="camera_depth_optical_frame">
-    <inertial>
-      <mass value="0.001" />
-      <inertia ixx="0.0001" ixy="0" ixz="0" iyy="0.0001" iyz="0" izz="0.0001" />
-    </inertial>
-  </link>
-  <joint name="camera_depth_optical_joint" type="fixed">
-    <parent link="camera_link" />
-    <child link="camera_depth_optical_frame" />
-    <origin xyz="0 -0.01 0" rpy="-1.570796 0 -1.570796" />
-  </joint> -->
 </robot>

File: panda_description/urdf/sensor_stick.gazebo.xacro (robot description, xacro)
@@ -4,55 +4,26 @@
   <gazebo reference="link_2"><material>Gazebo/White</material></gazebo>
   <gazebo reference="camera_base_link"><material>Gazebo/Grey</material></gazebo>
-  <gazebo reference="camera_mount_link">
-      <sensor name="d435_color" type="camera">
-        <always_on>1</always_on>
-        <update_rate>30</update_rate>
-        <visualize>1</visualize>
-        <pose>0 0.0175 0.0 0 -0 0</pose>
-        <topic>/color_camera</topic>
-        <camera name="d435">
-          <horizontal_fov>1.21126</horizontal_fov>
-          <image>
-            <width>640</width>
-            <height>480</height>
-            <format>RGB_INT8</format>
-          </image>
-          <clip>
-            <near>0.1</near>
-            <far>100</far>
-          </clip>
-          <noise>
-            <type>gaussian</type>
-            <mean>0</mean>
-            <stddev>0.007</stddev>
-          </noise>
-        </camera>
-      </sensor>
-      <sensor name='d435_depth' type='depth_camera'>
-        <always_on>1</always_on>
-        <update_rate>15</update_rate>
-        <visualize>1</visualize>
-        <topic>/depth_camera</topic>
-        <pose>0 0.04 -0.04 0 0 0</pose>
-        <camera name='d435'>
-          <horizontal_fov>1.48702</horizontal_fov>
-          <image>
-            <width>1280</width>
-            <height>720</height>
-          </image>
-          <clip>
-            <near>0.2</near>
-            <far>5</far>
-          </clip>
-          <noise>
-            <type>gaussian</type>
-            <mean>0</mean>
-            <stddev>0.1</stddev>
-          </noise>
-        </camera>
-        <plugin filename="libgz-sim-sensors-system.so" name="gz::sim::systems::Sensors">
-          <render_engine>ogre</render_engine>
-        </plugin>
-      </sensor>
-    </gazebo>
+<gazebo reference="camera_link">
+  <sensor name="my_rgbd_camera" type="rgbd_camera">
+    <plugin
+      filename="gz-sim-sensors-system"
+      name="gz::sim::systems::Sensors">
+      <render_engine>ogre2</render_engine>
+    </plugin>
+    <topic>/camera</topic>
+    <update_rate>30</update_rate>
+    <visualize>true</visualize>
+    <camera>
+      <horizontal_fov>1.047</horizontal_fov>
+      <image>
+        <width>640</width>
+        <height>480</height>
+      </image>
+      <clip>
+        <near>0.1</near>
+        <far>10</far>
+      </clip>
+    </camera>
+  </sensor>
+</gazebo>
 </robot>
